File: keyboards/Keyboard/Keyboard.kicad_pcb (KiCad board)
At the start: 2 copper layers, 96 parts, among them U1 RP2040_Zero, U2 RP2040_Zero, U3 TRRS, U4 TRRS

Commit message: add PCB routing, Mounting Hole
Parts:
- added H1: Mounting_Hole, MountingHole:MountingHole_2.2mm_M2, F.Cu at (19.1, 38.1)
- added H10: Mounting_Hole, MountingHole:MountingHole_2.2mm_M2, F.Cu at (304.2, 38.1)
- added H2: Mounting_Hole, MountingHole:MountingHole_2.2mm_M2, F.Cu at (19.1, 95.2)
- added H3: Mounting_Hole, MountingHole:MountingHole_2.2mm_M2, F.Cu at (152.4, 38.1)
- added H4: Mounting_Hole, MountingHole:MountingHole_2.2mm_M2, F.Cu at (152.4, 114.3)
- added H5: Mounting_Hole, MountingHole:MountingHole_2.2mm_M2, F.Cu at (76.2, 104.8)
- added H6: Mounting_Hole, MountingHole:MountingHole_2.2mm_M2, F.Cu at (247.1, 104.8)
- added H7: Mounting_Hole, MountingHole:MountingHole_2.2mm_M2, F.Cu at (170.9, 114.3)
- added H8: Mounting_Hole, MountingHole:MountingHole_2.2mm_M2, F.Cu at (170.9, 38.1)
- added H9: Mounting_Hole, MountingHole:MountingHole_2.2mm_M2, F.Cu at (304.2, 95.2)
- moved D26 5.32 mm to (228.0, 41.0)
- moved D32 5.32 mm to (228.0, 60.0)
- moved D39 5.32 mm to (228.0, 79.1)
- moved D46 5.32 mm to (228.0, 98.1)
- moved S36 5.32 mm to (180.4, 85.7)
- moved S43 5.32 mm to (180.4, 104.8)
- moved D24 5.32 mm to (189.9, 50.5)
- moved D25 5.32 mm to (209.0, 45.7)
- moved D27 5.32 mm to (247.1, 45.7)
- moved D28 5.32 mm to (266.1, 50.5)
- moved D29 5.32 mm to (285.2, 50.5)
- moved D30 5.32 mm to (189.9, 69.5)
- moved D31 5.32 mm to (209.0, 64.8)
- moved D33 5.32 mm to (247.1, 64.8)
- moved D34 5.32 mm to (266.1, 69.5)
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Connections:
- U1 pad 11: ROW3_Left -> unconnected-(U1-10-Pad11)
- U1 pad 12: ROW2_Left -> unconnected-(U1-11-Pad12)
- U1 pad 13: ROW1_Left -> unconnected-(U1-12-Pad13)
- U1 pad 14: ROW0_Left -> unconnected-(U1-13-Pad14)
- U1 pad 16: unconnected-(U1-15-Pad16) -> ROW3_Left
- U1 pad 17: unconnected-(U1-26-Pad17) -> ROW2_Left
- U1 pad 18: unconnected-(U1-27-Pad18) -> ROW1_Left
- U1 pad 19: unconnected-(U1-28-Pad19) -> ROW0_Left
- U2 pad 10: ROW0_Right -> unconnected-(U2-9-Pad10)
- U2 pad 11: ROW1_Right -> unconnected-(U2-10-Pad11)
- U2 pad 12: ROW2_Right -> unconnected-(U2-11-Pad12)
- U2 pad 13: ROW3_Right -> unconnected-(U2-12-Pad13)
- U2 pad 15: COL5_Right -> COL0_Right
- U2 pad 16: COL4_Right -> COL1_Right
- U2 pad 17: COL3_Right -> COL2_Right
- U2 pad 18: COL2_Right -> COL3_Right
- U2 pad 19: COL1_Right -> COL4_Right
- U2 pad 20: COL0_Right -> COL5_Right
- U2 pad 4: unconnected-(U2-3-Pad4) -> ROW0_Right
- U2 pad 5: unconnected-(U2-4-Pad5) -> ROW1_Right
- U2 pad 6: unconnected-(U2-5-Pad6) -> ROW2_Right
- U2 pad 7: unconnected-(U2-6-Pad7) -> ROW3_Right
Routing:
- net COL0_Left: track 38.1 -> 182.9 mm
- net COL5_Right: track 38.1 -> 175.9 mm
- net ROW2_Right: track 0.00 -> 137.4 mm
- net ROW2_Left: track 0.00 -> 135.0 mm
- net COL1_Left: track 81.4 -> 207.8 mm
- net COL4_Right: track 80.1 -> 201.1 mm
- net ROW1_Right: track 0.00 -> 120.8 mm
- net ROW1_Left: track 0.00 -> 119.1 mm
- net ROW3_Right: track 0.00 -> 118.9 mm
- net ROW3_Left: track 0.00 -> 116.5 mm
- net ROW0_Left: track 0.00 -> 112.9 mm
- net ROW0_Right: track 0.00 -> 110.1 mm
- net COL2_Left: track 84.1 -> 191.5 mm
- net COL3_Right: track 86.0 -> 187.7 mm
- net COL3_Left: track 90.5 -> 179.8 mm
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
Commit message: keyboard pcb design complete
Parts:
- moved S29 14.8 mm to (283.4, 38.1)
- moved S35 14.8 mm to (283.4, 57.1)
- moved S42 14.8 mm to (283.4, 76.2)
- moved S38 14.8 mm to (207.2, 71.4)
- moved S45 14.8 mm to (207.2, 90.5)
- moved S25 14.8 mm to (207.2, 33.3)
- moved S31 14.8 mm to (207.2, 52.4)
- moved D36 14.8 mm to (159.5, 79.1)
- moved D43 14.8 mm to (159.5, 98.1)
- moved H7 14.8 mm to (159.5, 104.8)
- moved D39 14.8 mm to (216.7, 69.5)
- moved D45 14.8 mm to (197.6, 93.3)
- moved D46 14.8 mm to (216.7, 88.6)
- moved H6 14.8 mm to (235.7, 95.2)
- moved H9 14.8 mm to (292.9, 85.7)
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Other:
- board outline added: 292.9 x 95.2 mm

Commit message: comlete pcb editing
Parts:
- added H11: Mounting_Hole, MountingHole:MountingHole_2.2mm_M2, F.Cu at (66.7, 19.1)
- added H12: Mounting_Hole, MountingHole:MountingHole_2.2mm_M2, F.Cu at (235.7, 19.1)
Routing:
- added copper zone on B.Cu, net (none)
- added copper zone on F.Cu, net (none)
Changed lines of the file:
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@@
     )
   )
+  (footprint "MountingHole:MountingHole_2.2mm_M2" (layer "F.Cu")
+    (at 66.675 19.05)
+    (descr "Mounting Hole 2.2mm, no annular, M2")
+    (tags "mounting hole 2.2mm no annular m2")
+    (property "Sheetfile" "Keyboard.kicad_sch")
+    (property "Sheetname" "")
+    (property "ki_description" "Mounting Hole without connection")
+    (property "ki_keywords" "mounting hole")
+    (attr exclude_from_pos_files)
+    (fp_text reference "H11" (at 0 -3.2) (layer "F.SilkS")
+        (effects (font (size 1 1) (thickness 0.15)))
+    )
+    (fp_text value "Mounting_Hole" (at 0 3.2) (layer "F.Fab")
+        (effects (font (size 1 1) (thickness 0.15)))
+    )
+    (fp_text user "${REFERENCE}" (at 0 0) (layer "F.Fab")
+        (effects (font (size 1 1) (thickness 0.15)))
+    )
+    (fp_circle (center 0 0) (end 2.2 0)
+      (stroke (width 0.15) (type solid)) (fill none) (layer "Cmts.User"))
+    (fp_circle (center 0 0) (end 2.45 0)
+      (stroke (width 0.05) (type solid)) (fill none) (layer "F.CrtYd"))
+    (pad "" np_thru_hole circle (at 0 0) (size 2.2 2.2) (drill 2.2) (layers "*.Cu" "*.Mask"))
+  )
   (footprint "ScottoKeebs_Components:TRRS_PJ-320A" (layer "F.Cu")
     (at 145.6375 61.9125 -90)
@@
     (pad "" np_thru_hole circle (at 0 0 180) (size 2.2 2.2) (drill 2.2) (layers "*.Cu" "*.Mask"))
   )
+  (footprint "MountingHole:MountingHole_2.2mm_M2" (layer "F.Cu")
+    (at 235.74375 19.05)
+    (descr "Mounting Hole 2.2mm, no annular, M2")
+    (tags "mounting hole 2.2mm no annular m2")
+    (property "Sheetfile" "Keyboard.kicad_sch")
+    (property "Sheetname" "")
+    (property "ki_description" "Mounting Hole without connection")
+    (property "ki_keywords" "mounting hole")
+    (attr exclude_from_pos_files)
+    (fp_text reference "H12" (at 0 -3.2) (layer "F.SilkS")
+        (effects (font (size 1 1) (thickness 0.15)))
+    )
+    (fp_text value "Mounting_Hole" (at 0 3.2) (layer "F.Fab")
+        (effects (font (size 1 1) (thickness 0.15)))
+    )
+    (fp_text user "${REFERENCE}" (at 0 0) (layer "F.Fab")
+        (effects (font (size 1 1) (thickness 0.15)))
+    )
+    (fp_circle (center 0 0) (end 2.2 0)
+      (stroke (width 0.15) (type solid)) (fill none) (layer "Cmts.User"))
+    (fp_circle (center 0 0) (end 2.45 0)
+      (stroke (width 0.05) (type solid)) (fill none) (layer "F.CrtYd"))
+    (pad "" np_thru_hole circle (at 0 0) (size 2.2 2.2) (drill 2.2) (layers "*.Cu" "*.Mask"))
+  )
   (footprint "ScottoKeebs_MX:MX_PCB_1.00u" (layer "F.Cu")
     (at 114.3 95.25)
@@
   (segment (start 168.63125 49.2) (end 157.21125 37.78) (width 0.25) (layer "F.Cu") (net 91))
   (segment (start 168.63125 63.6625) (end 168.63125 49.2) (width 0.25) (layer "F.Cu") (net 91))
+  (zone (net 0) (net_name "") (layers "F&B.Cu") (hatch edge 0.5)
+    (connect_pads (clearance 0.5))
+    (min_thickness 0.25) (filled_areas_thickness no)
+    (fill yes (thermal_gap 0.5) (thermal_bridge_width 0.5) (island_removal_mode 1) (island_area_min 10))
+    (polygon
+      (pts
+        (xy -7.14375 -2.38125)
+        (xy 300.0375 0)
+        (xy 300.0375 114.3)
+        (xy -4.7625 116.68125)
+      )
+    )
+  )
 )

Commit message: edit pcb file
Parts:
- added H13: Mounting_Hole, MountingHole:MountingHole_2.2mm_M2, F.Cu at (66.7, 19.1)
- added H14: Mounting_Hole, MountingHole:MountingHole_2.2mm_M2, F.Cu at (235.7, 19.1)
- added H15: Mounting_Hole, MountingHole:MountingHole_2.2mm_M2, F.Cu at (178.6, 26.2)
- added H16: Mounting_Hole, MountingHole:MountingHole_2.2mm_M2, F.Cu at (123.8, 26.2)
- moved H3 58.0 mm to (123.8, 85.7)
- moved H8 58.0 mm to (178.6, 85.7)
- moved H11 47.6 mm to (28.6, 47.6)
- moved H12 47.6 mm to (273.8, 47.6)
Routing:
- net COL4_Right: track 201.1 -> 203.9 mm
- net COL5_Right: track 175.9 -> 178.1 mm
- net COL3_Right: track 187.7 -> 189.4 mm
- net COL1_Right: track 148.9 -> 147.5 mm
- net COL0_Right: track 101.2 -> 99.9 mm
- net COL4_Left: track 156.6 -> 157.8 mm
Other:
- outline, holes or cut-outs redrawn
- board text added: "S5cene46-RP2040 ver.1.0 github.com/Jangmyun"
