File: keyboards/sceneOrtho/sceneOrtho.kicad_pcb (KiCad board)
At the start: 2 copper layers, 128 parts, among them J1 USB_C_Receptacle_USB2.0, J2 Conn_01x04, J3 Conn_01x05, U1 RP2040, U2 XC6206PxxxMR, U3 SRV05-4, U4 W25Q128JVS, Y1 Crystal_GND24

Commit message: .
Parts:
- added C13: 100n, Capacitor_SMD:C_0402_1005Metric, B.Cu at (73.5, 49.7)
- added C14: 100n, Capacitor_SMD:C_0402_1005Metric, B.Cu at (80.4, 49.6)
- added C15: 100n, Capacitor_SMD:C_0402_1005Metric, B.Cu at (72.7, 50.5)
- added C16: 100n, Capacitor_SMD:C_0402_1005Metric, B.Cu at (71.4, 54.0)
- moved J3 129.0 mm to (51.3, 48.4), turned to -90 degrees
- moved F1 127.3 mm to (33.3, 60.1), turned to -90 degrees
- moved C1 99.0 mm to (59.8, 54.8)
- moved C2 96.4 mm to (65.1, 57.1), turned to 90 degrees
- moved U2 95.4 mm to (61.9, 57.1)
- moved R4 86.3 mm to (65.6, 52.6), turned to 0 degrees
- moved U4 85.8 mm to (92.9, 50.8)
- moved R5 84.8 mm to (65.6, 54.0), turned to 0 degrees
- moved C12 79.4 mm to (84.1, 53.2), turned to -45 degrees
- moved R7 70.0 mm to (122.5, 56.2)
- moved BOOT1 69.1 mm to (129.4, 54.0)
- moved R8 69.1 mm to (122.7, 51.6)
- moved R9 69.1 mm to (122.7, 53.6)
- moved RST1 63.7 mm to (106.4, 56.0)
- moved R3 62.2 mm to (101.6, 58.2), turned to -90 degrees
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Connections:
- C12 pad 1: +5V -> +3V3
- C2 pad 1: +5V -> +3V3
- C3 pad 1: +5V -> +3V3
- C6 pad 1: +5V -> +3V3
- C7 pad 1: +5V -> +3V3
- C8 pad 1: +5V -> +3V3
- C9 pad 1: +5V -> +3V3
- J3 pad 1: RESET -> SWC
- J3 pad 2: +5V -> SWD
- J3 pad 3: GND -> RESET
- J3 pad 4: SWC -> +3V3
- J3 pad 5: SWD -> GND
- R3 pad 2: +5V -> +3V3
- R9 pad 2: +5V -> +3V3
- U1 pad 1: +5V -> +3V3
- U1 pad 10: +5V -> +3V3
- U1 pad 22: +5V -> +3V3
- U1 pad 33: +5V -> +3V3
- U1 pad 42: +5V -> +3V3
- U1 pad 43: +5V -> +3V3
- U1 pad 44: +5V -> +3V3
- U1 pad 48: +5V -> +3V3
- U1 pad 49: +5V -> +3V3
- U2 pad 2: +5V -> +3V3
- U4 pad 8: +5V -> +3V3
Routing:
- net GND: track 0.00 -> 139.0 mm, vias 0 -> 14
- net RESET: track 0.00 -> 105.4 mm, vias 0 -> 2
- net +3V3: track 0.00 -> 96.3 mm, vias 0 -> 1
- net D+: track 0.00 -> 50.7 mm
- net D-: track 0.00 -> 50.2 mm
- net +5V: track 0.00 -> 47.7 mm
- net SWC: track 0.00 -> 42.3 mm, vias 0 -> 1
- net SWD: track 0.00 -> 39.7 mm, vias 0 -> 1
- net VBUS: track 0.00 -> 13.4 mm
- net Q_IO3: track 0.00 -> 13.4 mm
- net Q_CLK: track 0.00 -> 12.0 mm
- net Q_IO0: track 0.00 -> 10.4 mm
- net Net-(U1-USB_DM): track 0.00 -> 10.1 mm
- net Net-(U1-USB_DP): track 0.00 -> 10.1 mm
- net XIN: track 0.00 -> 8.78 mm
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- added copper zone on B.Cu, net GND
- added copper zone on F.Cu, net GND
Other:
- board outline added: 227 x 90.5 mm
