File: keyboards/sceneOrtho/sceneOrtho.kicad_sch (KiCad schematic)
At the start: 128 parts, among them J1 USB_C_Receptacle_USB2.0, J2 Conn_01x04, J3 Conn_01x05, U1 RP2040, U2 XC6206PxxxMR, U3 SRV05-4, U4 W25Q128JVS, Y1 Crystal_GND24

Commit message: .
Parts:
- added C13, C14, C15, C16: 100n, Capacitor_SMD:C_0402_1005Metric, symbol Device:C_Small
Connections:
- net +1V1: now also C13.1
- net +5V: no longer C12.1, C2.1, C3.1, C6.1, C7.1, C8.1, C9.1, J3.2 (Pin_2), R3.2, R9.2, U1.1 (IOVDD), U1.10 (IOVDD), U1.22 (IOVDD), U1.33 (IOVDD), U1.42 (IOVDD), U1.43 (ADC_AVDD), U1.44 (VREG_IN), U1.48 (USB_VDD), U1.49 (IOVDD), U2.2 (VO), U4.8 (VCC)
- net GND: now also J3.5 (Pin_5), C13.2, C14.2, C15.2, C16.2; no longer J3.3 (Pin_3)
- net RESET: now also J3.3 (Pin_3); no longer J3.1 (Pin_1)
- net SWC: now also J3.1 (Pin_1); no longer J3.4 (Pin_4)
- net SWD: now also J3.2 (Pin_2); no longer J3.5 (Pin_5)
- new net +3V3: C12.1, C14.1, C15.1, C16.1, C2.1, C3.1, C6.1, C7.1, C8.1, C9.1, J3.4 (Pin_4), R3.2, R9.2, U1.1 (IOVDD), U1.10 (IOVDD), U1.22 (IOVDD), U1.33 (IOVDD), U1.42 (IOVDD), U1.43 (ADC_AVDD), U1.44 (VREG_IN), U1.48 (USB_VDD), U1.49 (IOVDD), U2.2 (VO), U4.8 (VCC)
Other:
- moved on the sheet: C3, C6, C7, C8, C9
