File: keyboards/SceneTax/SceneTax.kicad_sch (KiCad schematic)
At the start: 128 parts

Commit message: .
Parts:
- added J1, J2: RJ45, Connector_RJ:RJ45_Amphenol_54602-x08_Horizontal, symbol Connector:RJ45
- S1, S10, S11, S12, S13, S14, S15, S16, S17, S18, S19, S2, S20, S21, S22, S23, S24, S25, S26, S27, S28, S29, S3, S30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: footprint (none) -> key-switches.pretty-main:SW_Gateron_LowProfile_THT_19mmgap
