File: keyboards/owt36/kicad/owt36.kicad_pcb (KiCad board)
At the start: 2 copper layers, 76 parts, among them SW1 Switch, SW2 SW_DPST, U1 Nice_Nano_V2

Commit message: owt36 pcb layout
Parts:
- added ?: , , F.Cu at (249.0, 101.0)
- added ?: , , F.Cu at (214.0, 110.0)
- added ?: , , F.Cu at (187.0, 81.0)
- added ?: , , F.Cu at (46.0, 101.0)
- added ?: , , F.Cu at (109.0, 81.0)
- added ?: , , F.Cu at (243.0, 63.0)
- added ?: , , F.Cu at (174.0, 130.0)
- added ?: , , F.Cu at (82.0, 110.0)
- added ?: , , F.Cu at (167.0, 115.0)
- added ?: , , F.Cu at (135.0, 80.0)
- added ?: , , F.Cu at (53.0, 64.0)
- added ?: , , F.Cu at (129.0, 115.0)
- added ?: , , F.Cu at (122.0, 130.0)
- added ?: , , F.Cu at (161.0, 80.0)
- SW1, SW2, U1: moved to B.Cu
- moved S23 167.0 mm to (252.2, 57.6), turned to 2 degrees
- moved S28 142.4 mm to (256.7, 77.8), turned to 2 degrees
- moved S22 141.8 mm to (231.7, 56.0), turned to 7 degrees
- moved S33 127.2 mm to (260.6, 96.8), turned to 2 degrees
- moved S27 120.0 mm to (235.3, 75.0), turned to 12 degrees
- moved S21 118.2 mm to (212.2, 57.9), turned to 12 degrees
- moved D11 116.7 mm to (34.8, 100.4), turned to 178 degrees
- moved D6 112.3 mm to (38.6, 81.4), turned to 178 degrees
- moved S32 111.2 mm to (239.2, 93.7), turned to 12 degrees
- moved D1 107.5 mm to (43.1, 61.2), turned to 178 degrees
- moved S31 104.6 mm to (220.1, 95.2), turned to 12 degrees
- moved S26 103.4 mm to (216.1, 76.6), turned to 12 degrees
- moved D16 101.5 mm to (78.7, 125.2), turned to 153 degrees
- moved S20 98.8 mm to (192.7, 69.1), turned to 15 degrees
- moved S25 97.7 mm to (196.8, 87.8), turned to 15 degrees
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Other:
- board outline added: 250.7 x 111.8 mm
